File: BMW_E30_Gauge_Cluster_Early_Model/BMW_E30_Early_Cluster_Nexus/BMW_E30_Early_Cluster_Nexus.kicad_pcb (KiCad board)
At the start: 2 copper layers, 356.8 x 150 mm, 27 parts, among them J1 C1 - Blue Connector, J2 C2 - White Connector, J3 C3 - Yellow Connector, J4 Conn_01x16_Pin, J5 Conn_01x19_Socket, U1 Temperature Gauge, U2 Fuel Gauge

Commit message: Layout Updates
Layout changes made after first laser cut board comparison.
Parts:
- moved R3 1.60 mm to (52.1, 151.6)
- moved LA12 1.25 mm to (349.8, 187.7)
- moved LA4 0.91 mm to (126.2, 187.7)
- moved LA9 0.58 mm to (289.3, 187.7)
- moved LA7 0.57 mm to (248.9, 187.7)
- moved LA5 0.50 mm to (146.8, 187.7)
- moved LA8 0.49 mm to (269.1, 187.7)
- moved LA17 0.48 mm to (207.5, 91.2)
- moved LA16 0.36 mm to (199.6, 74.0)
- moved LA18 0.35 mm to (215.6, 74.0)
- moved U2 0.35 mm to (62.3, 162.0)
- moved LA20 0.18 mm to (374.6, 151.9)
- moved LA14 0.13 mm to (42.7, 150.4)
- moved U1 0.09 mm to (353.6, 162.0)
Routing:
- net Net-(U2-Vcc): track 5.95 -> 15.8 mm
- net Temp_gauge: track 202.9 -> 208.0 mm
- net Fuel_level: track 265.0 -> 269.2 mm
- net +12 T15: track 903.4 -> 906.6 mm, vias 2 -> 1
- net GNDPWR: track 858.1 -> 857.7 mm, vias 6 -> 3
- net Oil_pressure_ind-: track 48.3 -> 48.4 mm, vias 1 -> 0
- net Low_Fuel_ind-: vias 1 -> 0
Other:
- outline, holes or cut-outs redrawn
