File: BMW_E30_Gauge_Cluster_Early_Model/BMW_E30_Early_Cluster_Nexus/BMW_E30_Early_Cluster_Nexus.kicad_pcb (KiCad board)
At the start: 2 copper layers, 356.8 x 150 mm, 27 parts, among them J1 C1 - Blue Connector, J2 C2 - White Connector, J3 C3 - Yellow Connector, J4 Conn_01x16_Pin, J5 Conn_01x19_Socket, U1 Temperature Gauge, U2 Fuel Gauge

Commit message: Silkscreen Updates
Other:
- board text added: "Glow Plug [Diesel]"
- board text added: "Trailer Indicators"
- board text removed: "Glow plug [Diesel]"
- board text removed: "Trailer indicators"
Changed lines of the file:
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@@
 		)
 	)
-	(gr_text "Glow plug [Diesel]"
+	(gr_text "Glow Plug [Diesel]"
 		(at 66.5 196 0)
 		(layer "F.SilkS")
@@
 		)
 	)
-	(gr_text "Trailer indicators"
+	(gr_text "Trailer Indicators"
 		(at 167.5 195.7 0)
 		(layer "F.SilkS")

Commit message: Nexus Layout Updates + Footprint Updates
Updated fuel gauge and temp gauge footprints to have their locating holes included. Also widened the mounting holes for both gauge footprints.

Layout:
Moved fuel gauge to the right by 1mm, moved blue connector down 1mm and left 0.5mm, moved white connector down 1mm.
Parts:
- U1: footprint BMW_Cluster_Connectors:Gauge_fuel_temp -> BMW_Cluster_Connectors:Gauge_Temp
- U2: footprint BMW_Cluster_Connectors:Gauge_fuel_temp -> BMW_Cluster_Connectors:Gauge_Fuel
- moved J1 1.12 mm to (335.5, 139.8)
- moved J2 1.00 mm to (80.5, 139.8)
- moved R3 0.93 mm to (53.0, 151.6)
- moved U2 0.28 mm to (62.8, 162.0)
Routing:
- net GNDPWR: track 859.4 -> 861.2 mm
- net +12 T15: track 906.1 -> 904.4 mm
- net RH_ind: track 196.2 -> 197.8 mm
- net Rear_fog_ind+: track 127.9 -> 126.9 mm
- net Park_brake_ind-: track 271.0 -> 270.0 mm
- net Fuel_rate_input: track 284.5 -> 283.6 mm
- net +12 T30: track 242.1 -> 241.2 mm
- net START: track 158.3 -> 157.4 mm
- net Charge_Ind+: track 30.4 -> 29.5 mm
- net +12 T15_ACC: track 287.6 -> 288.3 mm
- net RAW_RPM_input: track 15.0 -> 14.3 mm
- net Net-(U2-Vcc): track 15.9 -> 15.3 mm
Other:
- outline, holes or cut-outs redrawn

Commit message: Standardized Board Location
Made board location the same as the late model project to make component locations easy to map between both projects.
Parts:
- moved J1 24.0 mm to (335.5, 163.8)
- moved J2 24.0 mm to (80.5, 163.8)
- moved J3 24.0 mm to (215.6, 206.5)
- moved J4 24.0 mm to (222.2, 126.9)
- moved J5 24.0 mm to (207.7, 215.5)
- moved JP1 24.0 mm to (229.0, 213.2)
- moved LA11 24.0 mm to (329.7, 213.0)
- moved LA12 24.0 mm to (349.8, 211.7)
- moved LA13a1 24.0 mm to (96.4, 197.4)
- moved LA13b1 24.0 mm to (319.8, 197.4)
- moved LA14 24.0 mm to (43.0, 174.0)
- moved LA15 24.0 mm to (208.0, 189.5)
- moved LA16 24.0 mm to (200.0, 98.0)
- moved LA17 24.0 mm to (208.0, 115.2)
- moved LA18 24.0 mm to (216.0, 98.0)
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