File: BMW_E30_Gauge_Cluster_Early_Model/BMW_E30_Early_Cluster_EG/BMW_E30_Early_Cluster_EG.kicad_sch (KiCad schematic)
At the start: 43 parts, among them J1 Conn_01x11_Socket, J2 To EG, Q1 BC547C, Q2 BC337, U1 4049, U2 4584, U3 LM2930-5.0_TO220, U4 LM2903, U5 SAJ300R, Y1 160 kHz

Commit message: EG Schematic Completed
Parts:
- removed C3: 47n, symbol Device:C
- removed C4: ?, symbol Device:C_Polarized
- removed C5: 2.2u, symbol Device:C_Polarized
- removed D4: 1N1418, Diode_THT:D_DO-34_SOD68_P10.16mm_Horizontal, symbol Diode:1N4005
- removed D5: BZX55C 18V, symbol Device:D_Zener
- removed MES1: Fuel Economy Gauge, symbol Device:Galvanometer
- removed Q2: BC337, Package_TO_SOT_THT:TO-92_Inline, symbol Transistor_BJT:BC337
- removed R14: 47k, Resistor_THT:R_Axial_DIN0207_L6.3mm_D2.5mm_P10.16mm_Horizontal, symbol Device:R
- removed R15: 120R, Resistor_THT:R_Axial_DIN0207_L6.3mm_D2.5mm_P10.16mm_Horizontal, symbol Device:R
- removed R16: 470k, Resistor_THT:R_Axial_DIN0207_L6.3mm_D2.5mm_P10.16mm_Horizontal, symbol Device:R
- removed R17: 100k, Resistor_THT:R_Axial_DIN0207_L6.3mm_D2.5mm_P10.16mm_Horizontal, symbol Device:R
- removed R18: 2k7, Resistor_THT:R_Axial_DIN0207_L6.3mm_D2.5mm_P10.16mm_Horizontal, symbol Device:R
- removed RN1: R2R_8B, Resistor_THT:R_Array_SIP8, symbol BMW_ICs:R2R_8B
- removed RV1, RV2: 220k, symbol Device:R_Potentiometer_Trim
- removed U1: 4049, Package_DIP:DIP-16_W7.62mm, symbol 4xxx:4049
- removed unit 3 of U2
- removed unit 2 of U4
- removed U5: SAJ300R, symbol BMW_ICs:SAJ300R
- removed Y1: 160 kHz, symbol Device:Crystal
- added U7: SCL4527B, symbol BMW_ICs:SCL4527B
Connections:
- net +5V: now also U7.16 (VDD), U7.3 (D)
- net GNDPWR: now also U7.10 (STROBE), U7.11 (INHBT_IN), U7.12 (CASCADE), U7.13 (CLR), U7.14 (A), U7.15 (B), U7.2 (C), U7.4 (SET_TO_"9"), U7.8 (VSS)
- net 4527_P9 renamed ~{Wheel_speed_filtered}
- net ~{Wheel_speed_filtered}: now also U7.9 (CLK)
- net PIC_P11 renamed Dist_pulse
- net PIC_P7 renamed Fuel_rate_filtered
- new net Wheel_speed_out: U7.6 (OUT)
- no-connect marks 14 -> 8
Other:
- added sheet Economy Gauge Driver (EG_Driver.kicad_sch)
- note added: "Connectors"
- note added: "Fuel Rate & Wheel Speed Signal Filtering"
- note added: "Power Filtering and Distribution"
- note added: "Unused Components/Pins"
- moved on the sheet: C1, C2, C6, D1, D2, D3, R10, R11, R12, R13, R2, R3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

Commit message: Layout Updates for EG
TODO: fix reference designators that were rewritten by accident. Original reference designators are listed in the schematic pdf.
Parts:
- Q1: footprint Package_TO_SOT_THT:TO-92_Inline -> Package_TO_SOT_THT:TO-92L_Wide
- R1: footprint (none) -> Resistor_THT:R_Axial_DIN0207_L6.3mm_D2.5mm_P10.16mm_Horizontal
- R2: footprint (none) -> Resistor_THT:R_Axial_DIN0309_L9.0mm_D3.2mm_P20.32mm_Horizontal
- U2: footprint (none) -> Package_DIP:DIP-14_W7.62mm_Socket_LongPads
- U5: renamed from U7; footprint (none) -> Package_DIP:DIP-16_W7.62mm_Socket_LongPads
- renumbered R8 to R10, R13 to R12, R12 to R13, R5 to R3, R3 to R4, R4 to R5, R9 to R6, R6 to R7, R7 to R8, R10 to R9, U3 to U7
