File: BMW_E30_Gauge_Cluster_Early_Model/BMW_E30_Early_Cluster_EG/BMW_E30_Early_Cluster_EG.kicad_sch (KiCad schematic)
At the start: 26 parts, among them J1 Conn_01x11_Socket, J2 To EG, Q1 BC547C, U2 4584, U4 LM2903, U5 SCL4527B, U7 LM2930-5.0_TO220

Commit message: EG Layout Updates
Parts:
- C1: footprint (none) -> Capacitor_THT:C_Disc_D3.0mm_W1.6mm_P2.50mm
- C2: footprint (none) -> Capacitor_THT:C_Rect_L13.0mm_W4.0mm_P10.00mm_FKS3_FKP3_MKS4
- C6: footprint (none) -> Capacitor_THT:CP_Radial_D8.0mm_P5.00mm
- renumbered R9 to R10, R13 to R12, R12 to R13, R4 to R3, R5 to R4, R3 to R5, R7 to R6, R8 to R7, R10 to R8, R6 to R9
Changed lines of the file:
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@@
 		(dnp no)
 		(fields_autoplaced yes)
-		(property "Reference" "R4"
+		(property "Reference" "R3"
 			(at 165.1 100.3299 0)
 			(effects
@@
 			(project "BMW_E30_Early_Cluster_EG"
 				(path "/b216cb44-2546-4a52-a541-225697d17737"
-					(reference "R4")
+					(reference "R3")
 					(unit 1)
 				)
@@
 			)
 		)
-		(property "Footprint" ""
+		(property "Footprint" "Capacitor_THT:C_Rect_L13.0mm_W4.0mm_P10.00mm_FKS3_FKP3_MKS4"
 			(at 207.9752 53.34 0)
 			(effects
@@
 		(dnp no)
 		(fields_autoplaced yes)
-		(property "Reference" "R7"
+		(property "Reference" "R6"
 			(at 190.5 93.9799 0)
 			(effects
@@
 			(project "BMW_E30_Early_Cluster_EG"
 				(path "/b216cb44-2546-4a52-a541-225697d17737"
-					(reference "R7")
+					(reference "R6")
 					(unit 1)
 				)
@@
 		(dnp no)
 		(fields_autoplaced yes)
-		(property "Reference" "R3"
+		(property "Reference" "R5"
 			(at 163.83 181.6099 0)
 			(effects
@@
 			(project "BMW_E30_Early_Cluster_EG"
 				(path "/b216cb44-2546-4a52-a541-225697d17737"
-					(reference "R3")
+					(reference "R5")
 					(unit 1)
 				)
@@
 		(dnp no)
 		(fields_autoplaced yes)
-		(property "Reference" "R6"
+		(property "Reference" "R9"
 			(at 175.26 182.88 90)
 			(effects
@@
 			(project "BMW_E30_Early_Cluster_EG"
 				(path "/b216cb44-2546-4a52-a541-225697d17737"
-					(reference "R6")
+					(reference "R9")
 					(unit 1)
 				)
@@
 		(dnp no)
 		(fields_autoplaced yes)
-		(property "Reference" "R12"
+		(property "Reference" "R13"
 			(at 231.14 107.9499 0)
 			(effects
@@
 			(project "BMW_E30_Early_Cluster_EG"
 				(path "/b216cb44-2546-4a52-a541-225697d17737"
-					(reference "R12")
+					(reference "R13")
 					(unit 1)
 				)
@@
 		(dnp no)
 		(fields_autoplaced yes)
-		(property "Reference" "R5"
+		(property "Reference" "R4"
 			(at 172.72 114.3 90)
 			(effects
@@
 			(project "BMW_E30_Early_Cluster_EG"
 				(path "/b216cb44-2546-4a52-a541-225697d17737"
-					(reference "R5")
+					(reference "R4")
 					(unit 1)
 				)
@@
 		(dnp no)
 		(fields_autoplaced yes)
-		(property "Reference" "R10"
+		(property "Reference" "R8"
 			(at 204.47 96.52 90)
 			(effects
@@
 			(project "BMW_E30_Early_Cluster_EG"
 				(path "/b216cb44-2546-4a52-a541-225697d17737"
-					(reference "R10")
+					(reference "R8")
 					(unit 1)
 				)
@@
 		(dnp no)
 		(fields_autoplaced yes)
-		(property "Reference" "R8"
+		(property "Reference" "R7"
 			(at 190.5 129.5399 0)
 			(effects
@@
 			(project "BMW_E30_Early_Cluster_EG"
 				(path "/b216cb44-2546-4a52-a541-225697d17737"
-					(reference "R8")
+					(reference "R7")
 					(unit 1)
 				)
@@
 		(dnp no)
 		(fields_autoplaced yes)
-		(property "Reference" "R13"
+		(property "Reference" "R12"
 			(at 248.92 111.76 90)
 			(effects
@@
 			(project "BMW_E30_Early_Cluster_EG"
 				(path "/b216cb44-2546-4a52-a541-225697d17737"
-					(reference "R13")
+					(reference "R12")
 					(unit 1)
 				)
@@
 			)
 		)
-		(property "Footprint" ""
+		(property "Footprint" "Capacitor_THT:C_Disc_D3.0mm_W1.6mm_P2.50mm"
 			(at 248.6152 53.34 0)
 			(effects
@@
 			)
 		)
-		(property "Footprint" ""
+		(property "Footprint" "Capacitor_THT:CP_Radial_D8.0mm_P5.00mm"
 			(at 195.2752 53.34 0)
 			(effects
@@
 		(dnp no)
 		(fields_autoplaced yes)
-		(property "Reference" "R9"
+		(property "Reference" "R10"
 			(at 190.5 196.8499 0)
 			(effects
@@
 			(project "BMW_E30_Early_Cluster_EG"
 				(path "/b216cb44-2546-4a52-a541-225697d17737"
-					(reference "R9")
+					(reference "R10")
 					(unit 1)
 				)

Commit message: EG Layout Updates
Added capacitor footprints and moved all resistors into place.
Parts:
- C1: footprint Capacitor_THT:C_Disc_D3.0mm_W1.6mm_P2.50mm -> Capacitor_THT:CP_Radial_Tantal_D5.0mm_P2.50mm
Changed lines of the file:
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@@
 			)
 		)
-		(property "Footprint" "Capacitor_THT:C_Disc_D3.0mm_W1.6mm_P2.50mm"
+		(property "Footprint" "Capacitor_THT:CP_Radial_Tantal_D5.0mm_P2.50mm"
 			(at 248.6152 53.34 0)
 			(effects

Commit message: Layout Updates for EG
Added footprints for J1 and J2 connectors. Also Changed footprint for RN1 to match original board. Next step is to route traces.
Parts:
- J1: footprint (none) -> BMW_Cluster_Connectors:ConnectorIV_EG_Socket
- J2: footprint (none) -> BMW_Cluster_Connectors:EG_Tach_Socket
Changed lines of the file:
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@@
 			)
 		)
-		(property "Footprint" ""
+		(property "Footprint" "BMW_Cluster_Connectors:ConnectorIV_EG_Socket"
 			(at 38.1 40.64 0)
 			(effects
@@
 			)
 		)
-		(property "Footprint" ""
+		(property "Footprint" "BMW_Cluster_Connectors:EG_Tach_Socket"
 			(at 38.1 87.63 0)
 			(effects

Commit message: Update Schematic PDFs
Other:
- company: Reagan Ansel -> Reans
Changed lines of the file:
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@@
 	(title_block
 		(title "BMW E30 Gauge Cluster Fuel Economy Gauge")
-		(company "Reagan Ansel")
-		(comment 1 "NOTE: All resistors are 5% tolorance unless otherwise noted")
+		(date "2026-06-03")
+		(company "Reans")
+		(comment 1 "Reagan Ansel")
+		(comment 2 "NOTE: All resistors are 5% tolorance unless otherwise noted")
 	)
 	(rectangle
@@
 		)
 		(instances
-			(project "BMW_E30_Early_Cluster_Tachometer"
+			(project "BMW_E30_Early_Cluster_EG"
 				(path "/b216cb44-2546-4a52-a541-225697d17737"
 					(reference "#PWR07")
@@
 		)
 		(instances
-			(project ""
+			(project "BMW_E30_Early_Cluster_EG"
 				(path "/b216cb44-2546-4a52-a541-225697d17737"
 					(reference "C2")
@@
 		)
 		(instances
-			(project "BMW_E30_Early_Cluster_Tachometer"
+			(project "BMW_E30_Early_Cluster_EG"
 				(path "/b216cb44-2546-4a52-a541-225697d17737"
 					(reference "#PWR012")
@@
 		)
 		(instances
-			(project ""
+			(project "BMW_E30_Early_Cluster_EG"
 				(path "/b216cb44-2546-4a52-a541-225697d17737"
 					(reference "J1")
@@
 		)
 		(instances
-			(project ""
+			(project "BMW_E30_Early_Cluster_EG"
 				(path "/b216cb44-2546-4a52-a541-225697d17737"
 					(reference "U5")
@@
 		)
 		(instances
-			(project ""
+			(project "BMW_E30_Early_Cluster_EG"
 				(path "/b216cb44-2546-4a52-a541-225697d17737"
 					(reference "U2")
@@
 		)
 		(instances
-			(project "BMW_E30_Early_Cluster_Tachometer"
+			(project "BMW_E30_Early_Cluster_EG"
 				(path "/b216cb44-2546-4a52-a541-225697d17737"
 					(reference "#PWR09")
@@
 		)
 		(instances
-			(project ""
+			(project "BMW_E30_Early_Cluster_EG"
 				(path "/b216cb44-2546-4a52-a541-225697d17737"
 					(reference "U2")
@@
 		)
 		(instances
-			(project ""
+			(project "BMW_E30_Early_Cluster_EG"
 				(path "/b216cb44-2546-4a52-a541-225697d17737"
 					(reference "D1")
@@
 		)
 		(instances
-			(project "BMW_E30_Early_Cluster_Tachometer"
+			(project "BMW_E30_Early_Cluster_EG"
 				(path "/b216cb44-2546-4a52-a541-225697d17737"
 					(reference "#PWR04")
@@
 		)
 		(instances
-			(project ""
+			(project "BMW_E30_Early_Cluster_EG"
 				(path "/b216cb44-2546-4a52-a541-225697d17737"
 					(reference "U2")
@@
 		)
 		(instances
-			(project "BMW_E30_Early_Cluster_Tachometer"
+			(project "BMW_E30_Early_Cluster_EG"
 				(path "/b216cb44-2546-4a52-a541-225697d17737"
 					(reference "R2")
@@
 		)
 		(instances
-			(project "BMW_E30_Early_Cluster_Tachometer"
+			(project "BMW_E30_Early_Cluster_EG"
 				(path "/b216cb44-2546-4a52-a541-225697d17737"
 					(reference "#PWR08")
@@
 		)
 		(instances
-			(project ""
+			(project "BMW_E30_Early_Cluster_EG"
 				(path "/b216cb44-2546-4a52-a541-225697d17737"
 					(reference "U4")
@@
 		)
 		(instances
-			(project "BMW_E30_Early_Cluster_Tachometer"
+			(project "BMW_E30_Early_Cluster_EG"
 				(path "/b216cb44-2546-4a52-a541-225697d17737"
 					(reference "#PWR06")
@@
 		)
 		(instances
-			(project ""
+			(project "BMW_E30_Early_Cluster_EG"
 				(path "/b216cb44-2546-4a52-a541-225697d17737"
 					(reference "R1")
@@
 		)
 		(instances
-			(project ""
+			(project "BMW_E30_Early_Cluster_EG"
 				(path "/b216cb44-2546-4a52-a541-225697d17737"
 					(reference "C1")
@@
 		)
 		(instances
-			(project ""
+			(project "BMW_E30_Early_Cluster_EG"
 				(path "/b216cb44-2546-4a52-a541-225697d17737"
 					(reference "J2")
@@
 		)
 		(instances
-			(project "BMW_E30_Early_Cluster_Tachometer"
+			(project "BMW_E30_Early_Cluster_EG"
 				(path "/b216cb44-2546-4a52-a541-225697d17737"
 					(reference "#PWR03")
@@
 		)
 		(instances
-			(project ""
+			(project "BMW_E30_Early_Cluster_EG"
 				(path "/b216cb44-2546-4a52-a541-225697d17737"
 					(reference "U7")
@@
 		)
 		(instances
-			(project ""
+			(project "BMW_E30_Early_Cluster_EG"
 				(path "/b216cb44-2546-4a52-a541-225697d17737"
 					(reference "U2")
@@
 		)
 		(instances
-			(project ""
+			(project "BMW_E30_Early_Cluster_EG"
 				(path "/b216cb44-2546-4a52-a541-225697d17737"
 					(reference "U2")
@@
 		)
 		(instances
-			(project ""
+			(project "BMW_E30_Early_Cluster_EG"
 				(path "/b216cb44-2546-4a52-a541-225697d17737"
 					(reference "U4")
@@
 		)
 		(instances
-			(project ""
+			(project "BMW_E30_Early_Cluster_EG"
 				(path "/b216cb44-2546-4a52-a541-225697d17737"
 					(reference "Q1")
@@
 		)
 		(instances
-			(project ""
+			(project "BMW_E30_Early_Cluster_EG"
 				(path "/b216cb44-2546-4a52-a541-225697d17737"
 					(reference "#PWR02")
@@
 		)
 		(instances
-			(project ""
+			(project "BMW_E30_Early_Cluster_EG"
 				(path "/b216cb44-2546-4a52-a541-225697d17737"
 					(reference "#PWR01")
@@
 		)
 		(instances
-			(project "BMW_E30_Early_Cluster_Tachometer"
+			(project "BMW_E30_Early_Cluster_EG"
 				(path "/b216cb44-2546-4a52-a541-225697d17737"
 					(reference "#PWR05")
@@
 	)
 	(embedded_fonts no)
+	(embedded_files
+		(file
+			(name "reans_sheet_template.kicad_wks")
+			(type worksheet)
+			(data |KLUv/WD/Cu0XAPbhaSEA1TZqxSYVNDoEMnCBWkUAFLHYT8LfLc64wmSW/n9CwQRfAFoAZABfTlM7
+				Cd4PPZP4H186+DUZmyftazMZJC2P8bFwUWq25kUL8mvHwkXR9pEtP+RPAAACHc97OanDZJkyfiu6
+				ZexMnfGD2a9nCIBAQaOUVnXWvtiW2T8EQKDkgCwiGFoOIdn/etgijP3Ss7lq001Ur56Xy2XSChD4
+				izG0r9ol7kx06g/5X/6a1VV7XqJQDq990Dues9+Mwx979pw4IR4v7ePbb9d8i9eDM9hT/3WSxGHt
+				2uJ1q+pJaX8GA4vQjuDbzqhJOcfXfePbr1LR9rtrPIGhJBC7qR8kM8Z09g4omXCSTTKynjjiS1u1
+				q3CTj080beoGpaw+TAqJdN6Eq1gUW6JrkAYXdfWk9EBhnWkl7tsUFo7ieR1p0Ah/UJFzFgWBwsys
+				itUDRWfNENlvxpauoBUjcUhlrs3u12aulxf0XKs+aBalZRWr16FaFa1zTkqrrWV11qovCsPoB+Ee
+				j0iCNBBdsEPihDapC6udeZCNyxjfJvk4juFpWkVZjw3CObqFDYCaoBFNhdgMSQqSFDLMAYBEhObI
+				NmZkXfEEgg31YlRO4GceOtZZSD4tPZJ8rJ74G8PkjH1JKkKawsKGheoJuP2+IlY18ntrNC2s74Pr
+				DVe+cSgd0L7HteZMeDaXmooSSh/c+bVoVTYLk6RKN7Cv2UoaCAZv6YCSS6nbIQTWD7UwQeis5W/V
+				g0dYgB5CyE6HNFbmmlkm5KySJ6yIRrRM5Uc4pc8u9BJFUDGI5kCOG6xadygVBOu2LFloyz3FUwK0
+				K2QvICvncQgSH7pSFluywCLJ0Rwlm2f0GkYN7sFxT4mPYCI2kaL4bSAlPOhlas5v4CmJJDLxSXKn
+				Odp9OHfwRZI7o8xhC2+Z4AAEWT5Rojog0dbMToQXcXHPsDoOuhAAXPmNnp2jRa7V/EUBa9S+lvzC
+				Ux9y2yG0bmId6AOKOjzjaHSplt4lCml0x3i3uxaxGR+0Cg==|
+			)
+			(checksum "582015C87F5C50DCCFBFE692861C814F")
+		)
+	)
 )
