File: BMW_E30_Gauge_Cluster_Early_Model/BMW_E30_Early_Cluster_EG/BMW_E30_Early_Cluster_EG.kicad_pcb (KiCad board)
At the start: 2 copper layers, 83.7 x 91.6 mm, 49 parts, among them J1 Conn_01x11_Socket, J2 To EG, Q1 BC547C, Q2 BC337, SW1 Coding Plug, U1 4049, U2 4584, U3 SAJ300R, U4 LM2903, U5 SCL4527B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

Commit message: Layout Updates
Routing:
- net VCC_T15: track 58.5 -> 180.9 mm
- net 6_cyl: track 9.28 -> 131.3 mm
- net Net-(D5-K): track 0.00 -> 99.2 mm
- net +5V: track 77.4 -> 159.4 mm, vias 2 -> 6
- net Net-(U3-M): track 0.00 -> 71.2 mm
- net GNDPWR: track 385.7 -> 455.4 mm
- net ~{Wheel_speed_filtered}: track 0.00 -> 58.6 mm, vias 0 -> 2
- net Net-(U4B-+): track 0.00 -> 55.4 mm
- net SW_02: track 0.00 -> 49.3 mm
- net SW_10: track 0.00 -> 41.6 mm
- net Net-(Q2-B): track 5.65 -> 44.8 mm
- net /Economy Gauge Driver/CLK: track 0.00 -> 36.0 mm, vias 0 -> 3
- net Wheel_speed_out: track 0.00 -> 35.1 mm, vias 0 -> 2
- net SW_09: track 0.00 -> 34.2 mm
- net Net-(Q2-E): track 0.00 -> 32.2 mm
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