File: BMW_E30_Gauge_Cluster_Early_Model/BMW_E30_Early_Cluster_Tachometer/BMW_E30_Early_Cluster_Tachometer.kicad_pcb (KiCad board)
At the start: 2 copper layers, 59.3 x 45.3 mm, 19 parts, among them J1 Conn_01x05_Pin, Q1 BC557, U1 SN29736P

Commit message: Tach Board Layout Complete
Parts:
- moved C2 0.30 mm to (134.8, 96.5)
Routing:
- net +12V T15: track 0.00 -> 157.5 mm, vias 0 -> 1
- net IC_P1: track 0.00 -> 142.7 mm
- net Net-(MES1--): track 0.00 -> 110.7 mm
- net Net-(U1-Cyl): track 0.00 -> 42.6 mm
- net IC_P6: track 0.00 -> 33.5 mm
- net IC_P2: track 0.00 -> 30.0 mm
- net Engine_spd_input: track 0.00 -> 29.2 mm
- net ~{6_cyl}: track 0.00 -> 16.8 mm
- net GNDPWR: track 0.00 -> 16.4 mm
- net Net-(Q1-B): track 0.00 -> 11.8 mm
- net Net-(C5-Pad1): track 0.00 -> 9.97 mm
- net Net-(Q1-C): track 0.00 -> 6.86 mm
- net Net-(R2-Pad2): track 0.00 -> 5.91 mm
- net Net-(R8-Pad1): track 0.00 -> 5.68 mm
Other:
- outline, holes or cut-outs redrawn
