File: BMW_E30_Gauge_Cluster_Early_Model/BMW_E30_Early_Cluster_Speedometer/BMW_E30_Early_Cluster_Speedometer.kicad_sch (KiCad schematic)
At the start: 37 parts, among them J1 Conn_01x06_Socket, J2 Conn_01x04_Socket, J3 To Hall effect board, M1 Odometer, Q1 BC327-40, Q2 BD135, U1 UAF2115

Commit message: Update Schematic PDFs
Other:
- company: Reagan Ansel -> Reans
Changed lines of the file:
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@@
 	(title_block
 		(title "BMW E30 Speedometer Driver Schematic")
-		(company "Reagan Ansel")
+		(date "2026-06-03")
+		(rev "0")
+		(company "Reans")
+		(comment 1 "Reagan Ansel")
 	)
 	(text "+12 V (Hot in accessory, run, or start) (+)"
@@
 		)
 		(instances
-			(project ""
+			(project "BMW_E30_Early_Cluster_Speedometer"
 				(path "/9a835706-2a71-4b4d-aadf-5c5569044960"
 					(reference "Q2")
@@
 		)
 		(instances
-			(project ""
+			(project "BMW_E30_Early_Cluster_Speedometer"
 				(path "/9a835706-2a71-4b4d-aadf-5c5569044960"
 					(reference "#PWR04")
@@
 		)
 		(instances
-			(project ""
+			(project "BMW_E30_Early_Cluster_Speedometer"
 				(path "/9a835706-2a71-4b4d-aadf-5c5569044960"
 					(reference "J3")
@@
 		)
 		(instances
-			(project ""
+			(project "BMW_E30_Early_Cluster_Speedometer"
 				(path "/9a835706-2a71-4b4d-aadf-5c5569044960"
 					(reference "U1")
@@
 		)
 		(instances
-			(project ""
+			(project "BMW_E30_Early_Cluster_Speedometer"
 				(path "/9a835706-2a71-4b4d-aadf-5c5569044960"
 					(reference "F1")
@@
 		)
 		(instances
-			(project ""
+			(project "BMW_E30_Early_Cluster_Speedometer"
 				(path "/9a835706-2a71-4b4d-aadf-5c5569044960"
 					(reference "D1")
@@
 		)
 		(instances
-			(project ""
+			(project "BMW_E30_Early_Cluster_Speedometer"
 				(path "/9a835706-2a71-4b4d-aadf-5c5569044960"
 					(reference "D6")
@@
 		)
 		(instances
-			(project ""
+			(project "BMW_E30_Early_Cluster_Speedometer"
 				(path "/9a835706-2a71-4b4d-aadf-5c5569044960"
 					(reference "C1")
@@
 		)
 		(instances
-			(project ""
+			(project "BMW_E30_Early_Cluster_Speedometer"
 				(path "/9a835706-2a71-4b4d-aadf-5c5569044960"
 					(reference "D2")
@@
 		)
 		(instances
-			(project ""
+			(project "BMW_E30_Early_Cluster_Speedometer"
 				(path "/9a835706-2a71-4b4d-aadf-5c5569044960"
 					(reference "#PWR01")
@@
 		)
 		(instances
-			(project ""
+			(project "BMW_E30_Early_Cluster_Speedometer"
 				(path "/9a835706-2a71-4b4d-aadf-5c5569044960"
 					(reference "MES1")
@@
 		)
 		(instances
-			(project ""
+			(project "BMW_E30_Early_Cluster_Speedometer"
 				(path "/9a835706-2a71-4b4d-aadf-5c5569044960"
 					(reference "J2")
@@
 		)
 		(instances
-			(project ""
+			(project "BMW_E30_Early_Cluster_Speedometer"
 				(path "/9a835706-2a71-4b4d-aadf-5c5569044960"
 					(reference "Q1")
@@
 		)
 		(instances
-			(project ""
+			(project "BMW_E30_Early_Cluster_Speedometer"
 				(path "/9a835706-2a71-4b4d-aadf-5c5569044960"
 					(reference "M1")
@@
 		)
 		(instances
-			(project ""
+			(project "BMW_E30_Early_Cluster_Speedometer"
 				(path "/9a835706-2a71-4b4d-aadf-5c5569044960"
 					(reference "R1")
@@
 		)
 		(instances
-			(project ""
+			(project "BMW_E30_Early_Cluster_Speedometer"
 				(path "/9a835706-2a71-4b4d-aadf-5c5569044960"
 					(reference "J1")
@@
 	)
 	(embedded_fonts no)
+	(embedded_files
+		(file
+			(name "reans_sheet_template.kicad_wks")
+			(type worksheet)
+			(data |KLUv/WD/Cu0XAPbhaSEA1TZqxSYVNDoEMnCBWkUAFLHYT8LfLc64wmSW/n9CwQRfAFoAZABfTlM7
+				Cd4PPZP4H186+DUZmyftazMZJC2P8bFwUWq25kUL8mvHwkXR9pEtP+RPAAACHc97OanDZJkyfiu6
+				ZexMnfGD2a9nCIBAQaOUVnXWvtiW2T8EQKDkgCwiGFoOIdn/etgijP3Ss7lq001Ur56Xy2XSChD4
+				izG0r9ol7kx06g/5X/6a1VV7XqJQDq990Dues9+Mwx979pw4IR4v7ePbb9d8i9eDM9hT/3WSxGHt
+				2uJ1q+pJaX8GA4vQjuDbzqhJOcfXfePbr1LR9rtrPIGhJBC7qR8kM8Z09g4omXCSTTKynjjiS1u1
+				q3CTj080beoGpaw+TAqJdN6Eq1gUW6JrkAYXdfWk9EBhnWkl7tsUFo7ieR1p0Ah/UJFzFgWBwsys
+				itUDRWfNENlvxpauoBUjcUhlrs3u12aulxf0XKs+aBalZRWr16FaFa1zTkqrrWV11qovCsPoB+Ee
+				j0iCNBBdsEPihDapC6udeZCNyxjfJvk4juFpWkVZjw3CObqFDYCaoBFNhdgMSQqSFDLMAYBEhObI
+				NmZkXfEEgg31YlRO4GceOtZZSD4tPZJ8rJ74G8PkjH1JKkKawsKGheoJuP2+IlY18ntrNC2s74Pr
+				DVe+cSgd0L7HteZMeDaXmooSSh/c+bVoVTYLk6RKN7Cv2UoaCAZv6YCSS6nbIQTWD7UwQeis5W/V
+				g0dYgB5CyE6HNFbmmlkm5KySJ6yIRrRM5Uc4pc8u9BJFUDGI5kCOG6xadygVBOu2LFloyz3FUwK0
+				K2QvICvncQgSH7pSFluywCLJ0Rwlm2f0GkYN7sFxT4mPYCI2kaL4bSAlPOhlas5v4CmJJDLxSXKn
+				Odp9OHfwRZI7o8xhC2+Z4AAEWT5Rojog0dbMToQXcXHPsDoOuhAAXPmNnp2jRa7V/EUBa9S+lvzC
+				Ux9y2yG0bmId6AOKOjzjaHSplt4lCml0x3i3uxaxGR+0Cg==|
+			)
+			(checksum "582015C87F5C50DCCFBFE692861C814F")
+		)
+	)
 )
