File: BMW_E30_Gauge_Cluster_Early_Model/BMW_E30_Early_Cluster_SI/BMW_E30_Early_Cluster_SI.kicad_sch (KiCad schematic)
At the start: 46 parts, among them J5 Nexus Connector, Q1 BC327-16, Q26 BC547B, U1 ITT SAF1093 MCU, Y1 Crystal

Commit message: Updates to Comparator Circuit
Updated Comparator circuit and the final pins of the MCU. Majority of signals and components are accounted for. Next step is footprint assignment and then double checking each component.
Parts:
- removed C3: 47u, symbol Device:C_Polarized_Small
- added R45: 750R, symbol Device:R
- added TP1, TP2, TP3, TP4, TP5, TP6: TestPoint_Alt, symbol Connector:TestPoint_Alt
Connections:
- net +5V: now also R45.2
- net at U1.10: now also TP2.1
- net at U1.26: now also TP3.1
- net at U1.27: now also TP4.1
- net at U1.29: now also TP5.1
- net at U1.36: now also R45.1, TP6.1
- net IC1_4: now reaches U1.4
- net at U1.9: now also TP1.1
Other:
- sheet Temperature Sensor ports: added batt_charge_state; removed none
- moved on the sheet: C11, D6, D7, R16, R32, R8, R9, U1, Y1
